Commit message: EDIT: mecanum_robot forward velocity change 1.5 -- > 5.5 and delete mecanum_slam_launch code

File: src/mecanum_robot_description/urdf/mecanum_robot/mecanum.gazebo.xacro (robot description, xacro)
@@ -37,5 +37,5 @@
   </xacro:macro>
   <xacro:macro name="sensor_gazebo" params="">
-    <!-- <gazebo reference="imu_link">
+    <gazebo reference="imu_link">
       <sensor type="imu" name="imu">
         <always_on>true</always_on>
@@ -71,5 +71,5 @@
         </imu>
       </plugin>
-    </gazebo> -->
+    </gazebo>
     <!-- <gazebo reference="front_R_wheel">
       <mu1>1.0</mu1>

File: src/mecanum_robot_description/urdf/mecanum_robot/mecanum_frame.urdf.xacro (robot description, xacro)
@@ -95,10 +95,10 @@
             </collision>
         </link>
-        <!-- <joint name="imu_joint" type="fixed">
+        <joint name="imu_joint" type="fixed">
           <parent link="base_link"/>
           <child link="imu_link"/>
           <origin xyz="0.0 0.0 0.10" rpy="0 0 0"/>
         </joint>
-        <link name="imu_link"/> -->
+        <link name="imu_link"/>
     </xacro:macro>
 </robot>
