Commit message: EDIT: MCL based python resampling code

File: src/mecanum_robot_description/urdf/mecanum_robot/mecanum_frame.urdf.xacro (robot description, xacro)
@@ -45,5 +45,5 @@
             </collision>
             <inertial>
-                <mass value="100.781" /> <!--20.781-->
+                <mass value="300.781" /> <!--20.781-->
                 <origin xyz="0.0 0.0 0.0" rpy="${pi/2} 0.0 ${-pi/2}"/>
                 <inertia ixx="3.9866734999999998" ixy="9.6705e-05"  ixz="0.000248215"  iyy="6.32225"  iyz="0.00284912"  izz="2.6884815" />

Commit message: EDIT: MCL based python resampling part

File: src/mecanum_robot_description/urdf/mecanum_robot/mecanum_frame.urdf.xacro (robot description, xacro)
@@ -45,5 +45,5 @@
             </collision>
             <inertial>
-                <mass value="300.781" /> <!--20.781-->
+                <mass value="50.781" /> <!--20.781-->
                 <origin xyz="0.0 0.0 0.0" rpy="${pi/2} 0.0 ${-pi/2}"/>
                 <inertia ixx="3.9866734999999998" ixy="9.6705e-05"  ixz="0.000248215"  iyy="6.32225"  iyz="0.00284912"  izz="2.6884815" />
